File: Hardware/pcb-rf-4g-ublox/Processor.sch (KiCad schematic (older format))
At the start: 43 parts, among them J4 Micro_SD_Card, J5 ST-LINK Connector, SW1 SW_SPDT, SW2 SW_Push_Dual, U3 AMS1117-3.3, U4 STM32F407VGTx

Commit message: Assign values to the components
Parts:
- C14, C16, C19, C20, C21, C22, C23, C24, C25, C26, C28, C29, C30, C31, C32, C33, C34, C35, C36, C40, C42, C43: value C -> 100nF
- C17: value C -> 10uF
- C27: value C -> 1000uF
- C37, C38: value C -> 4.7uF
- C39, C41: value C -> 1uF
- C44, C45: value C -> 2.2uF
- R10, R5, R6, R7, R8, R9: value R_Small -> 22E
- R13: value R -> 10K
